File: LDO_Stable_JAFWAK/LDO_Stable_JAFWAK.kicad_sch (KiCad schematic)
At the start: 20 parts, among them J1 VIN_DC, J15 VOUT_BUFF, J17 VS_BUFF, J2 VOUT, J24 Load Cell and Buffer, J3 GND, J4 GND, J6 AD_PINS, J8 VIN_FG

Commit message: Save current PCB project
Other:
- sheet Temp Sensor ports: added VS_BUFF; removed VIN
Changed lines of the file:
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@@
 		)
 	)
-	(global_label "VIN"
+	(global_label "VS_BUFF"
 		(shape input)
 		(at 116.84 140.97 0)
@@
 		)
 		(property "Intersheetrefs" "${INTERSHEET_REFS}"
-			(at 122.8491 140.97 0)
+			(at 127.8686 140.97 0)
 			(hide yes)
 			(show_name no)
@@
 		(in_pos_files yes)
 		(dnp no)
-		(fields_autoplaced yes)
 		(property "Reference" "#PWR050"
 			(at 74.93 143.51 0)
@@
 		)
 		(property "Value" "GND"
-			(at 74.93 142.24 0)
+			(at 78.232 138.176 0)
 			(show_name no)
 			(do_not_autoplace no)
@@
 			)
 		)
-		(pin "VIN" input
+		(pin "VS_BUFF" input
 			(at 114.3 140.97 0)
 			(effects
