File: LDO_Stable_JAFWAK/ldo_harness.kicad_sch (KiCad schematic)
At the start: 25 parts, among them J14 VOUT, J16 VDD_SEL, J22 IN_S, J23 VREF, J25 VIN, U1 SU272AFJK_LDO, U3 FXLP34, U6 FXLP34

Commit message: Roughed In schematic
Parts:
- removed J14: VOUT, TPS7A7001_Evaluation_Board_footprint_lib:SAMTEC_SMA-J-P-H-ST-TH1, symbol JAFWAK:SMA_FivePin
- removed J22: IN_S, TPS7A7001_Evaluation_Board_footprint_lib:SAMTEC_SMA-J-P-H-ST-TH1, symbol SMA-J-P-H-ST-TH1:SMA-J-P-H-ST-TH1
- removed J23: VREF, TPS7A7001_Evaluation_Board_footprint_lib:SAMTEC_SMA-J-P-H-ST-TH1, symbol JAFWAK:SMA_FivePin
- removed J25: VIN, TPS7A7001_Evaluation_Board_footprint_lib:SAMTEC_SMA-J-P-H-ST-TH1, symbol JAFWAK:SMA_FivePin
- removed JP1: PEC03SAAN, TPS7A7001_Evaluation_Board_footprint_lib:CONN_PEC03SAAN_SUL, symbol PEC03SAAN:PEC03SAAN
- removed U3: FXLP34, Package_LCC:PLCC-84_29.3x29.3mm_P1.27mm, symbol JAFWAK:FXLP34
- added J12: EN_FG, TPS7A7001_Evaluation_Board_footprint_lib:SAMTEC_SMA-J-P-H-ST-TH1, symbol JAFWAK:SMA_FivePin
- added J18: EN_SEL, Connector_PinHeader_2.54mm:PinHeader_2x08_P2.54mm_Vertical, symbol Connector_Generic:Conn_02x08_Odd_Even
- added J5: EN_AIN_SEL, Connector_PinHeader_2.54mm:PinHeader_2x04_P2.54mm_Vertical, symbol Connector_Generic:Conn_02x04_Odd_Even
- added R30: 0, Resistor_SMD:R_0805_2012Metric_Pad1.20x1.40mm_HandSolder, symbol Device:R
- added TP12: ~{EN_IN}, TPS7A7001_Evaluation_Board_footprint_lib:KEYSTONE_5016, symbol Connector:TestPoint
- added TP13: EN_IN, TPS7A7001_Evaluation_Board_footprint_lib:KEYSTONE_5016, symbol Connector:TestPoint
- added U8: FXLP34, Package_TO_SOT_SMD:SOT-353_SC-70-5, symbol JAFWAK:FXLP34
- C7: value C -> 1nF; footprint (none) -> Capacitor_SMD:C_0805_2012Metric_Pad1.18x1.45mm_HandSolder
- JP10: footprint TPS7A7001_Evaluation_Board_footprint_lib:CONN_PxC02S_SUL -> Connector_PinHeader_2.54mm:PinHeader_1x02_P2.54mm_Vertical
- TP1: value IN_S1 -> INA; footprint Keystone 5016 testpoint:KEYSTONE_5016 -> TPS7A7001_Evaluation_Board_footprint_lib:KEYSTONE_5016
- TP10: footprint Keystone 5016 testpoint:KEYSTONE_5016 -> TPS7A7001_Evaluation_Board_footprint_lib:KEYSTONE_5016
- TP2: value IN_S2 -> INB; footprint Keystone 5016 testpoint:KEYSTONE_5016 -> TPS7A7001_Evaluation_Board_footprint_lib:KEYSTONE_5016
- TP3: value OUT_S1 -> OUTB; footprint Keystone 5016 testpoint:KEYSTONE_5016 -> TPS7A7001_Evaluation_Board_footprint_lib:KEYSTONE_5016
- TP4: value OUT_S2 -> OUTA; footprint Keystone 5016 testpoint:KEYSTONE_5016 -> TPS7A7001_Evaluation_Board_footprint_lib:KEYSTONE_5016
- TP9: value EN -> EN_AIN; footprint Keystone 5016 testpoint:KEYSTONE_5016 -> TPS7A7001_Evaluation_Board_footprint_lib:KEYSTONE_5016
- U6: footprint (none) -> Package_TO_SOT_SMD:SOT-353_SC-70-5
Connections:
- net VIN is gone; now on net INA: R9.1, TP1.1
- net GND: now also U6.3 (GND), J12.2 (Ext), J12.3 (Ext), J12.4 (Ext), J12.5 (Ext), J18.12 (Pin_12), J18.2 (Pin_2), J5.3 (Pin_3), U8.3 (GND)
- net INB: now reaches J16.11 (Pin_11), J16.15 (Pin_15), J16.3 (Pin_3), J16.7 (Pin_7), R9.2, TP2.1
- net INB: now also R30.2; no longer C1.1, C2.1, C3.1
- net EN_OUT: now reaches U1.4 (EN_OUT)
- net EN_OUT: now also J18.16 (Pin_16)
- net ~{EN_OUT}: now reaches U1.5 (~{EN_OUT})
- net ~{EN_OUT}: now also J18.8 (Pin_8)
- net ~{EN_IN}: now reaches U1.6 (~{EN_IN})
- net ~{EN_IN}: now also J18.1 (Pin_1), J18.3 (Pin_3), J18.5 (Pin_5), J18.7 (Pin_7), TP12.1
- net EN_IN: now reaches U1.7 (EN_IN)
- net EN_IN: now also J18.11 (Pin_11), J18.13 (Pin_13), J18.15 (Pin_15), J18.9 (Pin_9), TP13.1
- net ADV: now reaches U6.1 (VCC1)
- net ADV: now also U8.1 (VCC1)
- net AD2: now reaches U6.2 (A)
- net AD2_SHIFT: now reaches U6.4 (Y)
- net AD2_SHIFT: now also J18.14 (Pin_14)
- net INA: now reaches U6.5 (VCC)
- net INA: now also J18.10 (Pin_10), J18.4 (Pin_4), J5.1 (Pin_1), U8.5 (VCC)
- net EN renamed EN_AIN
- net EN_AIN: now also J5.2 (Pin_2), J5.4 (Pin_4), J5.6 (Pin_6), J5.8 (Pin_8)
- net LDO_VOUT renamed OUTA
- net VOUT renamed OUTB
- new net: J12.1 (In), J5.5 (Pin_5)
- new net: C1.1, C2.1, C3.1, R30.1
- new net AD1: U8.2 (A)
- new net AD1_SHIFT: J18.6 (Pin_6), J5.7 (Pin_7), U8.4 (Y)
Other:
- note added: "Depopulate if you cant drive Vin with enough swing"
- note removed: "Need an ~{EN} signal from the input here?"
- note removed: "Select parts for Level shifting the Discovery"
- moved on the sheet: C1, C2, C3, C7, JP10, R14, R28, R29, R9, TP1, TP10, TP2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

Commit message: Started Layout
Other:
- moved on the sheet: J16

Commit message: Save current PCB project
Connections:
- new net EP: U1.33 (EP)
Changed lines of the file:
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@@
+		)
+	)
+	(label "EP"
+		(at 167.64 110.49 0)
+		(effects
+			(font
+				(size 1.27 1.27)
+			)
+			(justify left bottom)
 		)
 	)
@@
 		(pin "18"
 		)
+		(pin "33"
+		)
 		(instances
