File: LDO_Stable_JAFWAK/buffer.kicad_sch (KiCad schematic)
At the start: 4 parts, among them U5 BUF634AIDR

Commit message: Roughed In schematic
Parts:
- C14: value 10uF -> 100n
- JP11: footprint TPS7A7001_Evaluation_Board_footprint_lib:CONN_PxC02S_SUL -> Connector_PinHeader_2.54mm:PinHeader_1x02_P2.54mm_Vertical
Changed lines of the file:
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@@
 			)
 		)
-		(property "Footprint" "TPS7A7001_Evaluation_Board_footprint_lib:CONN_PxC02S_SUL"
+		(property "Footprint" "Connector_PinHeader_2.54mm:PinHeader_1x02_P2.54mm_Vertical"
 			(at 101.6 92.71 0)
 			(hide yes)
@@
 		(fields_autoplaced yes)
 		(property "Reference" "C14"
-			(at 161.29 91.4401 0)
-			(show_name no)
-			(do_not_autoplace no)
-			(effects
-				(font
-					(size 1.27 1.27)
-				)
-				(justify left)
-			)
-		)
-		(property "Value" "10uF"
-			(at 161.29 88.9001 0)
-			(show_name no)
-			(do_not_autoplace no)
-			(effects
-				(font
-					(size 1.27 1.27)
-				)
-				(justify left)
-			)
-		)
+			(at 168.91 88.8999 0)
+			(show_name no)
+			(do_not_autoplace no)
+			(effects
+				(font
+					(size 1.27 1.27)
+				)
+				(justify right)
+			)
+		)
+		(property "Value" "100n"
+			(at 168.91 91.4399 0)
+			(show_name no)
+			(do_not_autoplace no)
+			(effects
+				(font
+					(size 1.27 1.27)
+				)
+				(justify right)
+			)
+		)

Commit message: Started Layout
Changed lines of the file:
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@@
 		(color 0 0 0 0)
 	)
+	(junction
+		(at 162.56 80.01)
+		(diameter 0)
+		(color 0 0 0 0)
+	)
 	(wire
 		(pts
@@
 	(wire
 		(pts
-			(xy 158.75 80.01) (xy 165.1 80.01)
+			(xy 158.75 80.01) (xy 162.56 80.01)
 		)
 		(stroke
@@
 		(pts
 			(xy 102.87 92.71) (xy 101.6 92.71)
+		)
+		(stroke
+			(width 0)
+			(type default)
+		)
+	)
+	(wire
+		(pts
+			(xy 162.56 80.01) (xy 165.1 80.01)
 		)
 		(stroke
@@
 					(unit 1)
 				)
+			)
+		)
+	)
+	(symbol
+		(lib_id "power:PWR_FLAG")
+		(at 162.56 80.01 0)
+		(unit 1)
+		(body_style 1)
+		(exclude_from_sim no)
+		(in_bom yes)
+		(on_board yes)
+		(in_pos_files yes)
+		(dnp no)
+		(fields_autoplaced yes)
+		(property "Reference" "#FLG08"
+			(at 162.56 78.105 0)
+			(hide yes)
+			(show_name no)
+			(do_not_autoplace no)
+			(effects
+				(font
+					(size 1.27 1.27)
+				)
+			)
+		)
+		(property "Value" "PWR_FLAG"
+			(at 162.56 74.93 0)
+			(show_name no)
+			(do_not_autoplace no)
+			(effects
+				(font
+					(size 1.27 1.27)
+				)
+			)
+		)
+		(property "Footprint" ""
+			(at 162.56 80.01 0)
+			(hide yes)
+			(show_name no)
+			(do_not_autoplace no)
+			(effects
+				(font
+					(size 1.27 1.27)
+				)
+			)
+		)
+		(property "Datasheet" ""
+			(at 162.56 80.01 0)
+			(hide yes)
+			(show_name no)
+			(do_not_autoplace no)
+			(effects
+				(font
+					(size 1.27 1.27)
+				)
+			)
+		)
+		(property "Description" "Special symbol for telling ERC where power comes from"
+			(at 162.56 80.01 0)
+			(hide yes)
+			(show_name no)
+			(do_not_autoplace no)
+			(effects
+				(font
+					(size 1.27 1.27)
+				)
+			)
+		)
+		(pin "1"
+		)
+		(instances
+			(project "LDO_Stable_JAFWAK"
+				(path "/e797984e-8841-4b55-a934-93c9429b6b10/0ae94381-59df-4e68-8d23-513c5f52eb32"
+					(reference "#FLG09")
+					(unit 1)
+				)
+				(path "/e797984e-8841-4b55-a934-93c9429b6b10/430cf972-ca51-446c-aa23-29866872bb88"
+					(reference "#FLG08")
+					(unit 1)
+				)

Commit message: Several Changes
Moved temp sensor closer to chip
Add silkscreen
Moved capacitors closer to chip
Parts:
- C14: KiLib_Generator (none) -> SMD_2terminal_chip_molded
- JP3: renamed from JP11; KiLib_Generator (none) -> connector/pin_header_socket
- R5: renamed from R12; KiLib_Generator (none) -> SMD_2terminal_chip_molded
- renumbered U5 to U4
Changed lines of the file:
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@@
 		(in_pos_files yes)
 		(dnp no)
-		(property "Reference" "JP11"
+		(property "Reference" "JP3"
 			(at 92.964 99.06 0)
 			(show_name no)
@@
 		)
 		(property "Distributer Link 2" ""
+			(at 101.6 92.71 0)
+			(hide yes)
+			(show_name no)
+			(do_not_autoplace no)
+			(effects
+				(font
+					(size 1.27 1.27)
+				)
+			)
+		)
+		(property "KiLib_Generator" "connector/pin_header_socket"
 			(at 101.6 92.71 0)
 			(hide yes)
@@
 			(project "LDO_Stable_JAFWAK"
 				(path "/e797984e-8841-4b55-a934-93c9429b6b10/0ae94381-59df-4e68-8d23-513c5f52eb32"
-					(reference "JP12")
+					(reference "JP1")
 					(unit 1)
 				)
 				(path "/e797984e-8841-4b55-a934-93c9429b6b10/430cf972-ca51-446c-aa23-29866872bb88"
-					(reference "JP11")
+					(reference "JP3")
 					(unit 1)
 				)
@@
 		(dnp no)
 		(fields_autoplaced yes)
-		(property "Reference" "U5"
+		(property "Reference" "U4"
 			(at 140.97 72.39 0)
 			(show_name no)
@@
 			(project "LDO_Stable_JAFWAK"
 				(path "/e797984e-8841-4b55-a934-93c9429b6b10/0ae94381-59df-4e68-8d23-513c5f52eb32"
-					(reference "U7")
+					(reference "U2")
 					(unit 1)
 				)
 				(path "/e797984e-8841-4b55-a934-93c9429b6b10/430cf972-ca51-446c-aa23-29866872bb88"
-					(reference "U5")
+					(reference "U4")
 					(unit 1)
 				)
@@
 			)
 		)
+		(property "KiLib_Generator" "SMD_2terminal_chip_molded"
+			(at 165.1 90.17 0)
+			(hide yes)
+			(show_name no)
+			(do_not_autoplace no)
+			(effects
+				(font
+					(size 1.27 1.27)
+				)
+			)
+		)
 		(pin "1"
 		)
@@
 			(project "LDO_Stable_JAFWAK"
 				(path "/e797984e-8841-4b55-a934-93c9429b6b10/0ae94381-59df-4e68-8d23-513c5f52eb32"
-					(reference "C15")
+					(reference "C8")
 					(unit 1)
 				)
@@
 		(in_pos_files yes)
 		(dnp no)
-		(property "Reference" "R12"
+		(property "Reference" "R5"
 			(at 105.156 98.806 90)
 			(show_name no)
@@
 		)
 		(property "Distrbuter Link 2" "https://www.mouser.com/en/ProductDetail/YAGEO/RC0805FR-0710KL?qs=7bY8808IzHq6vrU3BeiiYw%3D%3D"
+			(at 102.87 99.06 0)
+			(hide yes)
+			(show_name no)
+			(do_not_autoplace no)
+			(effects
+				(font
+					(size 1.27 1.27)
+				)
+			)
+		)
+		(property "KiLib_Generator" "SMD_2terminal_chip_molded"
 			(at 102.87 99.06 0)
 			(hide yes)
@@
 			(project "LDO_Stable_JAFWAK"
 				(path "/e797984e-8841-4b55-a934-93c9429b6b10/0ae94381-59df-4e68-8d23-513c5f52eb32"
-					(reference "R13")
+					(reference "R3")
 					(unit 1)
 				)
 				(path "/e797984e-8841-4b55-a934-93c9429b6b10/430cf972-ca51-446c-aa23-29866872bb88"
-					(reference "R12")
-					(unit 1)
-				)
+					(reference "R5")
+					(unit 1)
+				)
