File: LDO_Stable_JAFWAK/load_cell.kicad_sch (KiCad schematic)
At the start: 16 parts, among them Q10 FDV305N, Q6 FDV305N, Q7 FDV305N, Q8 FDV305N, Q9 FDV305N

Commit message: Several Changes
Moved temp sensor closer to chip
Add silkscreen
Moved capacitors closer to chip
Parts:
- Q1: renamed from Q10; footprint FDV305N:SOT95P240X111-3N -> Package_TO_SOT_SMD:TSOT-23
- Q2: renamed from Q9; footprint FDV305N:SOT95P240X111-3N -> Package_TO_SOT_SMD:TSOT-23
- Q3: renamed from Q8; footprint FDV305N:SOT95P240X111-3N -> Package_TO_SOT_SMD:TSOT-23
- Q4: renamed from Q7; footprint FDV305N:SOT95P240X111-3N -> Package_TO_SOT_SMD:TSOT-23
- Q5: renamed from Q6; footprint FDV305N:SOT95P240X111-3N -> Package_TO_SOT_SMD:TSOT-23
- R10: renamed from R20; KiLib_Generator (none) -> SMD_2terminal_chip_molded
- R11: renamed from R18; KiLib_Generator (none) -> SMD_2terminal_chip_molded
- R12: renamed from R16; KiLib_Generator (none) -> SMD_2terminal_chip_molded
- R15: renamed from R26; KiLib_Generator (none) -> SMD_2terminal_chip_molded
- R16: renamed from R25; KiLib_Generator (none) -> SMD_2terminal_chip_molded
- R17: renamed from R24; KiLib_Generator (none) -> SMD_2terminal_chip_molded
- R18: renamed from R22; KiLib_Generator (none) -> SMD_2terminal_chip_molded
- R19: KiLib_Generator (none) -> SMD_2terminal_chip_molded
- R20: renamed from R17; KiLib_Generator (none) -> SMD_2terminal_chip_molded
- R8: renamed from R23; KiLib_Generator (none) -> SMD_2terminal_chip_molded
- R9: renamed from R21; KiLib_Generator (none) -> SMD_2terminal_chip_molded
Changed lines of the file:
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@@
+			)
+		)
+		(property "KiLib_Generator" "SMD_2terminal_chip_molded"
+			(at 113.03 68.58 0)
+			(hide yes)
+			(show_name no)
+			(do_not_autoplace no)
+			(effects
+				(font
+					(size 1.27 1.27)
+				)
 			)
 		)
@@
 		(dnp no)
 		(fields_autoplaced yes)
-		(property "Reference" "R18"
+		(property "Reference" "R11"
 			(at 105.41 114.2999 0)
 			(show_name no)
@@
 		)
 		(property "Distributer Link 2" "https://www.mouser.com/en/ProductDetail/YAGEO/RC0805FR-0710KL?qs=7bY8808IzHq6vrU3BeiiYw%3D%3D"
+			(at 102.87 115.57 0)
+			(hide yes)
+			(show_name no)
+			(do_not_autoplace no)
+			(effects
+				(font
+					(size 1.27 1.27)
+				)
+			)
+		)
+		(property "KiLib_Generator" "SMD_2terminal_chip_molded"
 			(at 102.87 115.57 0)
 			(hide yes)
@@
 			(project "LDO_Stable_JAFWAK"
 				(path "/e797984e-8841-4b55-a934-93c9429b6b10/dc9a158e-4ee1-42ad-aacb-b9976914ef03"
-					(reference "R18")
+					(reference "R11")
 					(unit 1)
 				)
@@
 		(dnp no)
 		(fields_autoplaced yes)
-		(property "Reference" "R25"
+		(property "Reference" "R16"
 			(at 158.75 67.3099 0)
 			(show_name no)
@@
 		)
 		(property "Distributer Link 2" ""
+			(at 156.21 68.58 0)
+			(hide yes)
+			(show_name no)
+			(do_not_autoplace no)
+			(effects
+				(font
+					(size 1.27 1.27)
+				)
+			)
+		)
+		(property "KiLib_Generator" "SMD_2terminal_chip_molded"
 			(at 156.21 68.58 0)
 			(hide yes)
@@
 			(project "LDO_Stable_JAFWAK"
 				(path "/e797984e-8841-4b55-a934-93c9429b6b10/dc9a158e-4ee1-42ad-aacb-b9976914ef03"
-					(reference "R25")
+					(reference "R16")
 					(unit 1)
 				)
@@
 		(dnp no)
 		(fields_autoplaced yes)
-		(property "Reference" "Q9"
+		(property "Reference" "Q2"
 			(at 160.02 77.4699 0)
 			(show_name no)
@@
 			)
 		)
-		(property "Footprint" "FDV305N:SOT95P240X111-3N"
+		(property "Footprint" "Package_TO_SOT_SMD:TSOT-23"
 			(at 153.67 78.74 0)
 			(hide yes)
@@
 			(project "LDO_Stable_JAFWAK"
 				(path "/e797984e-8841-4b55-a934-93c9429b6b10/dc9a158e-4ee1-42ad-aacb-b9976914ef03"
-					(reference "Q9")
+					(reference "Q2")
 					(unit 1)
 				)
@@
 		(dnp no)
 		(fields_autoplaced yes)
-		(property "Reference" "R22"
+		(property "Reference" "R18"
 			(at 129.54 67.3099 0)
 			(show_name no)
@@
 		)
 		(property "Distributer Link 2" ""
+			(at 127 68.58 0)
+			(hide yes)
+			(show_name no)
+			(do_not_autoplace no)
+			(effects
+				(font
+					(size 1.27 1.27)
+				)
+			)
+		)
+		(property "KiLib_Generator" "SMD_2terminal_chip_molded"
 			(at 127 68.58 0)
 			(hide yes)
@@
 			(project "LDO_Stable_JAFWAK"
 				(path "/e797984e-8841-4b55-a934-93c9429b6b10/dc9a158e-4ee1-42ad-aacb-b9976914ef03"
-					(reference "R22")
+					(reference "R18")
 					(unit 1)
 				)
@@
 		(dnp no)
 		(fields_autoplaced yes)
-		(property "Reference" "Q8"
+		(property "Reference" "Q3"
 			(at 137.16 77.4699 0)
 			(show_name no)
@@
 			)
 		)
-		(property "Footprint" "FDV305N:SOT95P240X111-3N"
+		(property "Footprint" "Package_TO_SOT_SMD:TSOT-23"
 			(at 130.81 78.74 0)
 			(hide yes)
@@
 			(project "LDO_Stable_JAFWAK"
 				(path "/e797984e-8841-4b55-a934-93c9429b6b10/dc9a158e-4ee1-42ad-aacb-b9976914ef03"
-					(reference "Q8")
+					(reference "Q3")
 					(unit 1)
 				)
@@
 		(dnp no)
 		(fields_autoplaced yes)
-		(property "Reference" "Q10"
+		(property "Reference" "Q1"
 			(at 180.34 77.4699 0)
 			(show_name no)
@@
 			)
 		)
-		(property "Footprint" "FDV305N:SOT95P240X111-3N"
+		(property "Footprint" "Package_TO_SOT_SMD:TSOT-23"
 			(at 173.99 78.74 0)
 			(hide yes)
@@
 			(project "LDO_Stable_JAFWAK"
 				(path "/e797984e-8841-4b55-a934-93c9429b6b10/dc9a158e-4ee1-42ad-aacb-b9976914ef03"
-					(reference "Q10")
+					(reference "Q1")
 					(unit 1)
 				)
@@
 		(dnp no)
 		(fields_autoplaced yes)
-		(property "Reference" "R23"
+		(property "Reference" "R8"
 			(at 139.7 114.2999 0)
 			(show_name no)
@@
 		)
 		(property "Distributer Link 2" "https://www.mouser.com/en/ProductDetail/YAGEO/RC0805FR-0710KL?qs=7bY8808IzHq6vrU3BeiiYw%3D%3D"
+			(at 137.16 115.57 0)
+			(hide yes)
+			(show_name no)
+			(do_not_autoplace no)
+			(effects
+				(font
+					(size 1.27 1.27)
+				)
+			)
+		)
+		(property "KiLib_Generator" "SMD_2terminal_chip_molded"
 			(at 137.16 115.57 0)
 			(hide yes)
@@
 			(project "LDO_Stable_JAFWAK"
 				(path "/e797984e-8841-4b55-a934-93c9429b6b10/dc9a158e-4ee1-42ad-aacb-b9976914ef03"
-					(reference "R23")
+					(reference "R8")
 					(unit 1)
 				)
@@
 		(dnp no)
 		(fields_autoplaced yes)
-		(property "Reference" "R17"
+		(property "Reference" "R20"
 			(at 93.98 67.3099 0)
 			(show_name no)
@@
 		)
 		(property "Distributer Link 2" "https://www.mouser.com/en/ProductDetail/TE-Connectivity-Holsworthy/RQ73C2A249RBTD?qs=gZXFycFWdAMgKEchKsVnjg%3D%3D"
+			(at 91.44 68.58 0)
+			(hide yes)
+			(show_name no)
+			(do_not_autoplace no)
+			(effects
+				(font
+					(size 1.27 1.27)
+				)
+			)
+		)
+		(property "KiLib_Generator" "SMD_2terminal_chip_molded"
 			(at 91.44 68.58 0)
 			(hide yes)
@@
 			(project "LDO_Stable_JAFWAK"
 				(path "/e797984e-8841-4b55-a934-93c9429b6b10/dc9a158e-4ee1-42ad-aacb-b9976914ef03"
-					(reference "R17")
+					(reference "R20")
 					(unit 1)
 				)
@@
 		(dnp no)
 		(fields_autoplaced yes)
-		(property "Reference" "Q7"
+		(property "Reference" "Q4"
 			(at 116.84 77.4699 0)
 			(show_name no)
@@
 			)
 		)
-		(property "Footprint" "FDV305N:SOT95P240X111-3N"
+		(property "Footprint" "Package_TO_SOT_SMD:TSOT-23"
 			(at 110.49 78.74 0)
 			(hide yes)
@@
 			(project "LDO_Stable_JAFWAK"
 				(path "/e797984e-8841-4b55-a934-93c9429b6b10/dc9a158e-4ee1-42ad-aacb-b9976914ef03"
-					(reference "Q7")
+					(reference "Q4")
 					(unit 1)
 				)
@@
 		(dnp no)
 		(fields_autoplaced yes)
-		(property "Reference" "R21"
+		(property "Reference" "R9"
 			(at 128.27 114.2999 0)
 			(show_name no)
@@
 		)
 		(property "Distributer Link 2" "https://www.mouser.com/en/ProductDetail/YAGEO/RC0805FR-0710KL?qs=7bY8808IzHq6vrU3BeiiYw%3D%3D"
+			(at 125.73 115.57 0)
+			(hide yes)
+			(show_name no)
+			(do_not_autoplace no)
+			(effects
+				(font
+					(size 1.27 1.27)
+				)
+			)
+		)
+		(property "KiLib_Generator" "SMD_2terminal_chip_molded"
 			(at 125.73 115.57 0)
 			(hide yes)
@@
 			(project "LDO_Stable_JAFWAK"
 				(path "/e797984e-8841-4b55-a934-93c9429b6b10/dc9a158e-4ee1-42ad-aacb-b9976914ef03"
-					(reference "R21")
+					(reference "R9")
 					(unit 1)
 				)
@@
 		(dnp no)
 		(fields_autoplaced yes)
-		(property "Reference" "Q6"
+		(property "Reference" "Q5"
 			(at 95.25 77.4699 0)
 			(show_name no)
@@
 			)
 		)
-		(property "Footprint" "FDV305N:SOT95P240X111-3N"
+		(property "Footprint" "Package_TO_SOT_SMD:TSOT-23"
 			(at 88.9 78.74 0)
 			(hide yes)
@@
 			(project "LDO_Stable_JAFWAK"
 				(path "/e797984e-8841-4b55-a934-93c9429b6b10/dc9a158e-4ee1-42ad-aacb-b9976914ef03"
-					(reference "Q6")
+					(reference "Q5")
 					(unit 1)
 				)
@@
 		(dnp no)
 		(fields_autoplaced yes)
-		(property "Reference" "R16"
+		(property "Reference" "R12"
 			(at 92.71 114.2999 0)
 			(show_name no)
@@
 		)
 		(property "Distributer Link 2" "https://www.mouser.com/en/ProductDetail/YAGEO/RC0805FR-0710KL?qs=7bY8808IzHq6vrU3BeiiYw%3D%3D"
+			(at 90.17 115.57 0)
+			(hide yes)
+			(show_name no)
+			(do_not_autoplace no)
+			(effects
+				(font
+					(size 1.27 1.27)
+				)
+			)
+		)
+		(property "KiLib_Generator" "SMD_2terminal_chip_molded"
 			(at 90.17 115.57 0)
 			(hide yes)
@@
 			(project "LDO_Stable_JAFWAK"
 				(path "/e797984e-8841-4b55-a934-93c9429b6b10/dc9a158e-4ee1-42ad-aacb-b9976914ef03"
-					(reference "R16")
+					(reference "R12")
 					(unit 1)
 				)
@@
 		(dnp no)
 		(fields_autoplaced yes)
-		(property "Reference" "R20"
+		(property "Reference" "R10"
 			(at 115.57 114.2999 0)
 			(show_name no)
@@
 		)
 		(property "Distributer Link 2" "https://www.mouser.com/en/ProductDetail/YAGEO/RC0805FR-0710KL?qs=7bY8808IzHq6vrU3BeiiYw%3D%3D"
+			(at 113.03 115.57 0)
+			(hide yes)
+			(show_name no)
+			(do_not_autoplace no)
+			(effects
+				(font
+					(size 1.27 1.27)
+				)
+			)
+		)
+		(property "KiLib_Generator" "SMD_2terminal_chip_molded"
 			(at 113.03 115.57 0)
 			(hide yes)
@@
 			(project "LDO_Stable_JAFWAK"
 				(path "/e797984e-8841-4b55-a934-93c9429b6b10/dc9a158e-4ee1-42ad-aacb-b9976914ef03"
-					(reference "R20")
+					(reference "R10")
 					(unit 1)
 				)
@@
 		(dnp no)
 		(fields_autoplaced yes)
-		(property "Reference" "R26"
+		(property "Reference" "R15"
 			(at 179.07 67.3099 0)
 			(show_name no)
@@
 		)
 		(property "Distributer Link 2" ""
+			(at 176.53 68.58 0)
+			(hide yes)
+			(show_name no)
+			(do_not_autoplace no)
+			(effects
+				(font
+					(size 1.27 1.27)
+				)
+			)
+		)
+		(property "KiLib_Generator" "SMD_2terminal_chip_molded"
 			(at 176.53 68.58 0)
 			(hide yes)
@@
 			(project "LDO_Stable_JAFWAK"
 				(path "/e797984e-8841-4b55-a934-93c9429b6b10/dc9a158e-4ee1-42ad-aacb-b9976914ef03"
-					(reference "R26")
+					(reference "R15")
 					(unit 1)
 				)
@@
 		(dnp no)
 		(fields_autoplaced yes)
-		(property "Reference" "R24"
+		(property "Reference" "R17"
 			(at 140.97 67.3099 0)
 			(show_name no)
@@
 		)
 		(property "Distributer Link 2" ""
+			(at 138.43 68.58 0)
+			(hide yes)
+			(show_name no)
+			(do_not_autoplace no)
+			(effects
+				(font
+					(size 1.27 1.27)
+				)
+			)
+		)
+		(property "KiLib_Generator" "SMD_2terminal_chip_molded"
 			(at 138.43 68.58 0)
 			(hide yes)
@@
 			(project "LDO_Stable_JAFWAK"
 				(path "/e797984e-8841-4b55-a934-93c9429b6b10/dc9a158e-4ee1-42ad-aacb-b9976914ef03"
-					(reference "R24")
+					(reference "R17")
 					(unit 1)
 				)
